File: Crystal.kicad_sch (KiCad schematic)
At the start: 13 parts, among them SW1 SW_Push, U1 HPM5E31IPB1, Y1 24Mhz

Commit message: finish
Parts:
- Y1: footprint Crystal:Crystal_SMD_3225-4Pin_3.2x2.5mm -> Crystal:Crystal_SMD_2016-4Pin_2.0x1.6mm
