File: HPM5E31.kicad_pcb (KiCad board)
At the start: 4 copper layers, 75 x 50 mm, 199 parts, among them J1 Conn_ARM_JTAG_SWD_10, J10 Conn_01x06_MountingPin, J11 Conn_01x03_Pin, J12 Conn_01x04_MountingPin, J13 Conn_01x06_MountingPin, J14 USB_C_Receptacle_USB2.0_16P, J15 Conn_01x03_Socket, J16 Conn_01x04_Socket, J2 Conn_01x03_MountingPin, J3 RJ45_Hanrun_HR911105A_Horizon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, J4 Conn_01x04_MountingPin, J5 Conn_01x03_Pin, J6 Conn_01x02_MountingPin, J7 Conn_01x06_MountingPin, J8 Conn_01x06_MountingPin, J9 Conn_01x06_MountingPin, Q1 SS8050, Q2 SS8050, SW1 SW_Push, U1 HPM5E31IPB1, U10 REF3033, U11 RY8411, U12 XC6210B332MR, U13 AFA11-S08GLA-00, U2 LAN8720A, U3 QS-301-AGS5P, U4 MLT-5020, U5 TJA1051TK-3, U6 RTL8211F-CG, U7 7*7*5-6P-L WX, U8 HR911130A, U9 USBLC6-2SC6, Y1 24Mhz, Y2 X322525MOB4SI, Y3 X322525MOB4SI

Commit message: 修改错误引脚
Parts:
- removed C37, C38, C39: 100nF, Capacitor_SMD:C_0603_1608Metric
- removed R13: 10K, Resistor_SMD:R_0603_1608Metric
- removed U3: QS-301-AGS5P, mylib:QS-301-AGS5P_C42377853
- added D10: LED, LED_SMD:LED_0603_1608Metric, F.Cu at (213.7, 64.6)
- added D12: LED, LED_SMD:LED_0603_1608Metric, F.Cu at (209.4, 67.7)
- added D13: LED, LED_SMD:LED_0603_1608Metric, F.Cu at (212.3, 67.7)
- added D14: LED, LED_SMD:LED_0603_1608Metric, F.Cu at (215.2, 67.7)
- added D9: LED, LED_SMD:LED_0603_1608Metric, F.Cu at (210.9, 64.6)
- added R66: 3.3K, Resistor_SMD:R_0603_1608Metric, F.Cu at (212.3, 64.6)
- added R67: 3.3K, Resistor_SMD:R_0603_1608Metric, F.Cu at (215.1, 64.6)
- added R68: 10K, Resistor_SMD:R_0603_1608Metric, F.Cu at (216.7, 67.7)
- L2, L3: value L -> 4.7uH
- moved C52 3.25 mm to (234.0, 90.0)
- moved C53 3.25 mm to (234.0, 91.4)
- moved C3 1.03 mm to (216.7, 92.1)
- moved C4 0.86 mm to (216.7, 93.3)
- moved R4 0.85 mm to (215.7, 85.4)
- moved R15 0.82 mm to (213.8, 67.7), turned to -90 degrees
- moved R3 0.79 mm to (215.7, 86.9)
- moved R14 0.72 mm to (210.9, 67.7), turned to -90 degrees
- moved C42 0.69 mm to (216.7, 94.5)
- moved C9 0.62 mm to (215.7, 84.1)
- moved L1 0.48 mm to (216.2, 89.5), turned to -90 degrees
- moved C7 0.34 mm to (216.2, 86.9)
- moved R2 0.23 mm to (216.1, 85.5)
Connections:
- L1 pad 2: +3.3V -> Net-(U1A-DCDC_LP)
- R14 pad 1: +3.3V -> /PIN_A/EMCODER_A
- R14 pad 2: /PIN_A/ENCODER_KEY -> Net-(D12-A)
- R15 pad 1: +3.3V -> /PIN_A/ENCODER_KEY
- R15 pad 2: /PIN_A/ENCODER_B -> Net-(D13-A)
- U1 pad 30: GND -> Net-(U1A-DCDC_LP)
- U1 pad 6: /PIN_A/BUZZER -> /PIN_A/LED
- U1 pad 7: /PIN_A/LED -> /PIN_A/BUZZER
Routing:
- net /PIN_A/ENCODER_B: track 61.0 -> 56.8 mm
- net Net-(C52-Pad2): track 4.68 -> 8.45 mm
- net Net-(U1A-DCDC_LP): track 0.00 -> 3.68 mm
- net Net-(U1A-DCDC_SNS): track 64.6 -> 68.2 mm, vias 8 -> 7
- net /PIN_A/ENCODER_KEY: track 58.2 -> 54.9 mm
- net /PIN_A/BUZZER: track 12.3 -> 14.7 mm
- net Net-(D12-A): track 0.00 -> 1.54 mm
- net Net-(D14-A): track 0.00 -> 1.47 mm
- net Net-(D13-A): track 0.00 -> 1.47 mm
- net /PIN_A/EMCODER_A: track 55.6 -> 54.1 mm
- net Net-(D9-A): track 0.00 -> 1.40 mm
- net Net-(D10-A): track 0.00 -> 1.40 mm
- net +3.3V: track 349.1 -> 350.3 mm
- net GND: track 127.0 -> 125.8 mm
- net /PIN_F/AVDD10: track 43.6 -> 42.4 mm
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- removed copper zone on F.Cu, net Net-(U1A-DCDC_SNS)
Other:
- board text added: "HPM5E31_V0.2"
- board text added: "X"
- board text removed: "HPM5E31_V0.1"
- board text removed: "x"
