File: PIN_F.kicad_sch (KiCad schematic)
At the start: 60 parts, among them J13 Conn_01x06_MountingPin, SW2 SW_DIP_x03, SW3 SW_DIP_x03, U1 HPM5E31IPB1, U6 RTL8211F-CG, U7 7*7*5-6P-L WX, U8 HR911130A, Y3 X322525MOB4SI

Commit message: finish
Parts:
- removed SW2, SW3: SW_DIP_x03, Button_Switch_SMD:SW_DIP_SPSTx03_Slide_KingTek_DSHP03TS_W7.62mm_P1.27mm, symbol Switch:SW_DIP_x03
- added C74: 10uF, Capacitor_SMD:C_0603_1608Metric, symbol Device:C
- added C75: 100nF, Capacitor_SMD:C_0603_1608Metric, symbol Device:C
- added D5, D6, D7, D8: ESD9B3.3ST5G, Diode_SMD:D_SOD-323, symbol Diode:ESD9B3.3ST5G
- added R55, R56, R57, R58, R59, R60: 4.7K, Resistor_SMD:R_0603_1608Metric, symbol Device:R
- Y3: footprint Crystal:Crystal_SMD_3225-4Pin_3.2x2.5mm -> Crystal:Crystal_SMD_2016-4Pin_2.0x1.6mm
Connections:
- net CFG\LDO0/LED1: now also C75.2, R56.1
- net CFG_EXT/LED0: now also R55.1
- net CFG_LDO1/LED2: now also C74.2, R57.1
- net GND: now also C74.1, C75.1, R55.2, R56.2, R57.2, R58.2, R59.2, R60.2
- net MDIN0: now also D8.2 (A2)
- net MDIN1: now also D7.2 (A2)
- net MDIN2: now also D6.2 (A2)
- net MDIN3: now also D5.2 (A2)
- net MDIP0: now also D8.1 (A1)
- net MDIP1: now also D7.1 (A1)
- net MDIP2: now also D6.1 (A1)
- net MDIP3: now also D5.1 (A1)
- net PLLOFF/RXD2: now also R58.1
- net RXDLY/RXD0: now also R60.1
- net TXDLY/RXD1: now also R59.1

Commit message: demo第一版
Parts:
- added R63, R64, R65: 4.7K, Resistor_SMD:R_0402_1005Metric, symbol Device:R
- added TP1, TP2, TP3: TestPoint, TestPoint:TestPoint_Pad_D1.0mm, symbol Connector:TestPoint
Connections:
- net +3.3V: now also TP1.1
- net ETH0.RXCK: now also R64.1
- net ETH0.RXD3: now also R65.1
- net ETH0.RXDV: now also R63.1
- net GND: now also R63.2, R65.2, TP3.1
- net VCC3V3_PHY: now also R64.2
- new net +5V: TP2.1
Other:
- note added: "PHY_ADDRES"
- moved on the sheet: C42, J13, U1D

Commit message: add pin description
Other:
- note removed: "PHY_ADDRES"
- moved on the sheet: C46, C47, C48, C49, C50, C51, C52, C53, C54, C55, C56, C57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

Commit message: 修改错误引脚
Parts:
- L2: value L -> 4.7uH
Changed lines of the file:
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@@
 			)
 		)
-		(property "Value" "L"
+		(property "Value" "4.7uH"
 			(at 257.81 156.21 90)
 			(show_name no)
